Commit message: Simulacion en Gazebo lista

File: humanoide_gazebo/urdf/humanoide_main.xacro (robot description, xacro)
@@ -120,5 +120,5 @@
      x = "0.0" y = "0.02" z = "0.01" parent = "link_servos_pierna_izquierda"
      gx = "-1" gy = "0" gz = "0"
-     child = "link_muslo_pierna_izquierda" effort = "8.4" velocity = "0.45"/>
+     child = "link_muslo_pierna_izquierda" effort = "55" velocity = "0.45"/>
      <!--Joint muslo izq - rodilla izq-->
     <xacro:joint_revoluta name="q3"

File: humanoide_gazebo/urdf/humanoide_meshes.xacro (robot description, xacro)
@@ -243,5 +243,5 @@
             <parent link="${parent}" />
             <axis rpy="0 0 0" xyz="${gx} ${gy} ${gz}" />
-            <limit effort="${effort}" lower="0" upper="${2*PI}" velocity="${velocity}"/>
+            <limit effort="${effort}" lower="${-2*PI}" upper="${2*PI}" velocity="${velocity}"/>
         </joint>
     </xacro:macro>

Commit message: Humanoide completo con IMU y camara

File: humanoide_gazebo/urdf/humanoide_main.xacro (robot description, xacro)
@@ -68,40 +68,40 @@
      x = "0.0" y = "0.0" z = "0.75" parent = "link_torso"
      gx = "0" gy = "0" gz = "1"
-     child = "link_cuello" effort = "2.5" velocity = "0.92"/>
+     child = "link_cuello" effort = "2.5" velocity = "5.76"/>
      <!--Joint cuello - cabeza-->
     <xacro:joint_revoluta name="q20"
      x = "0.0" y = "0.0" z = "0.02" parent = "link_cuello"
      gx = "-1" gy = "0" gz = "0"
-     child = "link_cabeza" effort = "2.5" velocity = "0.92"/>
+     child = "link_cabeza" effort = "2.5" velocity = "5.76"/>
     <!--Joint Torso - hombro izquierdo-->
     <xacro:joint_revoluta name="q13"
      x = "-0.11" y = "0.0" z = "0.7" parent = "link_torso"
      gx = "-1" gy = "0" gz = "0"
-     child = "link_hombro_izq" effort = "2.5" velocity = "0.92"/>
+     child = "link_hombro_izq" effort = "2.5" velocity = "5.76"/>
     <!--joint hombro izquierdo - Brazo izquierdo-->
     <xacro:joint_revoluta name="q14"
      x = "-0.03" y = "0.0" z = "0.01" parent = "link_hombro_izq"
      gx = "0" gy = "-1" gz = "0"
-     child = "link_brazo_izquierdo" effort = "2.5" velocity = "0.92"/>
+     child = "link_brazo_izquierdo" effort = "2.5" velocity = "5.76"/>
      <!--joint Brazo izquierdo - palmal izquierdo-->
     <xacro:joint_revoluta name="q15"
      x = "0.0" y = "0.0" z = "-0.2" parent = "link_brazo_izquierdo"
      gx = "0" gy = "1" gz = "0"
-     child = "link_palma_izquierdo" effort = "2.5" velocity = "0.92"/>
+     child = "link_palma_izquierdo" effort = "2.5" velocity = "5.76"/>
     <!--Joint Torso - hombro derecho-->
     <xacro:joint_revoluta name="q16"
      x = "0.11" y = "0.0" z = "0.7" parent = "link_torso"
      gx = "1" gy = "0" gz = "0"
-     child = "link_hombro_der" effort = "2.5" velocity = "0.92"/>
+     child = "link_hombro_der" effort = "2.5" velocity = "5.76"/>
     <!--joint hombro derecho - Brazo derecho-->
     <xacro:joint_revoluta name="q17"
      x = "0.03" y = "0.0" z = "0.01" parent = "link_hombro_der"
      gx = "0" gy = "-1" gz = "0"
-     child = "link_brazo_derecho" effort = "2.5" velocity = "0.92"/>
+     child = "link_brazo_derecho" effort = "2.5" velocity = "5.76"/>
      <!--joint Brazo derecho - palma derecho-->
     <xacro:joint_revoluta name="q18"
      x = "0.0" y = "0.0" z = "-0.2" parent = "link_brazo_derecho"
      gx = "0" gy = "1" gz = "0"
-     child = "link_palma_derecho" effort = "2.5" velocity = "0.92"/>
+     child = "link_palma_derecho" effort = "2.5" velocity = "5.76"/>
     <!--Joint Torso - metal pierna izquierda X-->
     <joint name="q6" type="fixed">
@@ -109,5 +109,5 @@
         <child link="link_metal_pierna_izquierda" />
         <parent link="link_torso" />
-        <limit effort="2.5" lower="0" upper="${2*PI}" velocity="0.92"/>
+        <limit effort="8.4" lower="0" upper="${2*PI}" velocity="5.76"/>
     </joint>
     <!--Joint metal pierna izquierdo - servos pierna izquierda X-->
@@ -115,25 +115,25 @@
      x = "0.0" y = "-0.02625" z = "-0.03" parent = "link_metal_pierna_izquierda"
      gx = "0" gy = "1" gz = "0"
-     child = "link_servos_pierna_izquierda" effort = "8.4" velocity = "0.45"/>
+     child = "link_servos_pierna_izquierda" effort = "8.4" velocity = "4.72"/>
      <!--Joint servos pierna izquierda - muslo izq-->
     <xacro:joint_revoluta name="q4"
      x = "0.0" y = "0.02" z = "0.01" parent = "link_servos_pierna_izquierda"
      gx = "-1" gy = "0" gz = "0"
-     child = "link_muslo_pierna_izquierda" effort = "55" velocity = "0.45"/>
+     child = "link_muslo_pierna_izquierda" effort = "8.4" velocity = "4.72"/>
      <!--Joint muslo izq - rodilla izq-->
     <xacro:joint_revoluta name="q3"
      x = "0.0" y = "0.0" z = "-0.2" parent = "link_muslo_pierna_izquierda"
      gx = "-1" gy = "0" gz = "0"
-     child = "link_rodilla_pierna_izquierda" effort = "8.4" velocity = "0.45"/>
+     child = "link_rodilla_pierna_izquierda" effort = "8.4" velocity = "4.72"/>
      <!--Joint rodilla izq - tob_izq-->
     <xacro:joint_revoluta name="q2"
      x = "0.0" y = "-0.0" z = "-0.16" parent = "link_rodilla_pierna_izquierda"
      gx = "1" gy = "0" gz = "0"
-     child = "link_servos_tob_pierna_izquierda" effort = "8.4" velocity = "0.45"/>
+     child = "link_servos_tob_pierna_izquierda" effort = "8.4" velocity = "4.72"/>
      <!--Joint tob_izq - pie izq-->
     <xacro:joint_revoluta name="q1"
      x = "0.0" y = "0.02625" z = "-0.025" parent = "link_servos_tob_pierna_izquierda"
      gx = "0" gy = "-1" gz = "0"
-     child = "link_pie_izq" effort = "8.4" velocity = "0.45"/>
+     child = "link_pie_izq" effort = "55" velocity = "4.72"/>
      <!--Joint Torso - metal pierna derechaX-->
     <joint name="q12" type="fixed">
@@ -141,5 +141,5 @@
         <child link="link_metal_pierna_derecha" />
         <parent link="link_torso" />
-        <limit effort="8.4" lower="0" upper="${2*PI}" velocity="0.45"/>
+        <limit effort="8.4" lower="0" upper="${2*PI}" velocity="4.72"/>
     </joint>
     <!--Joint metal pierna derecha - servos pierna derecha X-->
@@ -147,25 +147,25 @@
      x = "0.0" y = "-0.02625" z = "-0.03" parent = "link_metal_pierna_derecha"
      gx = "0" gy = "1" gz = "0"
-     child = "link_servos_pierna_derecha" effort = "8.4" velocity = "0.45"/>
+     child = "link_servos_pierna_derecha" effort = "8.4" velocity = "4.72"/>
      <!--Joint servos pierna derecha - muslo der-->
     <xacro:joint_revoluta name="q10"
      x = "0.0" y = "0.02" z = "0.01" parent = "link_servos_pierna_derecha"
      gx = "1" gy = "0" gz = "0"
-     child = "link_muslo_pierna_derecha" effort = "8.4" velocity = "0.45"/>
+     child = "link_muslo_pierna_derecha" effort = "8.4" velocity = "4.72"/>
      <!--Joint muslo der - rodilla der-->
     <xacro:joint_revoluta name="q9"
      x = "0.0" y = "0.0" z = "-0.2" parent = "link_muslo_pierna_derecha"
      gx = "1" gy = "0" gz = "0"
-     child = "link_rodilla_pierna_derecha" effort = "8.4" velocity = "0.45"/>
+     child = "link_rodilla_pierna_derecha" effort = "8.4" velocity = "4.72"/>
      <!--Joint rodilla der - tob_der-->
     <xacro:joint_revoluta name="q8"
      x = "0.0" y = "0.0" z = "-0.16" parent = "link_rodilla_pierna_derecha"
      gx = "-1" gy = "0" gz = "0"
-     child = "link_servos_tob_pierna_derecha" effort = "8.4" velocity = "0.45"/>
+     child = "link_servos_tob_pierna_derecha" effort = "8.4" velocity = "4.72"/>
      <!--Joint tob_der - pie der-->
     <xacro:joint_revoluta name="q7"
      x = "0.0" y = "0.02625" z = "-0.025" parent = "link_servos_tob_pierna_derecha"
      gx = "0" gy = "-1" gz = "0"
-     child = "link_pie_der" effort = "8.4" velocity = "0.45"/>
+     child = "link_pie_der" effort = "8.4" velocity = "4.72"/>
     <!--Transmisiones-->
     <gazebo>
@@ -192,3 +192,32 @@
     <xacro:MX_28T name = "q19_trans" motor_name = "motor_q19" joint_name = "q19"/>
     <xacro:MX_28T name = "q20_trans" motor_name = "motor_q20" joint_name = "q20"/>
+    <joint name="camera_joint" type="fixed">
+    <axis xyz="0 1 0" />
+        <origin xyz="0.0 0.025 0.05" rpy="0 0 ${PI/2}"/>
+        <parent link="link_cabeza"/>
+        <child link="camera_link"/>
+    </joint>
+    <!-- Camera -->
+    <link name="camera_link">
+        <collision>
+            <origin xyz="0 0 0" rpy="0 0 0"/>
+            <geometry>
+                <box size="0.005 0.005 0.005"/>
+            </geometry>
+        </collision>
+        <visual>
+            <origin xyz="0 0 0" rpy="0 0 0"/>
+            <geometry>
+                <box size="0.005 0.005 0.005"/>
+            </geometry>
+            <material name="red"/>
+        </visual>
+        <inertial>
+            <mass value="1e-5" />
+            <origin xyz="0 0 0" rpy="0 0 0"/>
+            <inertia ixx="1e-6" ixy="0" ixz="0" iyy="1e-6" iyz="0" izz="1e-6" />
+        </inertial>
+    </link>
+    <xacro:camera_cabeza name="camera_link"/>
+    <xacro:IMU_torsro name="link_torso"/>
 </robot>

File: humanoide_gazebo/urdf/humanoide_meshes.xacro (robot description, xacro)
@@ -247,8 +247,66 @@
     </xacro:macro>
     <!-- ROS Control plugin for Gazebo -->
-    <gazebo>
-        <plugin name="gazebo_ros_control" filename="libgazebo_ros_control.so">
-        <robotNamespace>/simple_model</robotNamespace>
-        </plugin>
-    </gazebo>
+    <xacro:macro name="camera_cabeza" params="name">
+        <gazebo reference="${name}">
+            <sensor type="camera" name="camera1">
+            <update_rate>30.0</update_rate>
+            <camera name="head">
+                <horizontal_fov>1.3962634</horizontal_fov>
+                <image>
+                <width>1280</width>
+                <height>720</height>
+                <format>R8G8B8</format>
+                </image>
+                <clip>
+                <near>0.02</near>
+                <far>300</far>
+                </clip>
+                <noise>
+                <type>gaussian</type>
+                <!-- Noise is sampled independently per pixel on each frame.
+                    That pixel's noise value is added to each of its color
+                    channels, which at that point lie in the range [0,1]. -->
+                <mean>0.0</mean>
+                <stddev>0.007</stddev>
+                </noise>
+            </camera>
+            <plugin name="camera_controller" filename="libgazebo_ros_camera.so">
+                <alwaysOn>true</alwaysOn>
+                <updateRate>0.0</updateRate>
+                <cameraName>Bogobot_model/camera1</cameraName>
+                <imageTopicName>image_raw</imageTopicName>
+                <cameraInfoTopicName>camera_info</cameraInfoTopicName>
+                <frameName>camera_link</frameName>
+                <hackBaseline>0.07</hackBaseline>
+                <distortionK1>0.0</distortionK1>
+                <distortionK2>0.0</distortionK2>
+                <distortionK3>0.0</distortionK3>
+                <distortionT1>0.0</distortionT1>
+                <distortionT2>0.0</distortionT2>
+            </plugin>
+            </sensor>
+        </gazebo>
+    </xacro:macro>
+    <xacro:macro name="IMU_torsro" params="name">
+        <gazebo reference="${name}">
+            <gravity>true</gravity>
+            <sensor name="imu_sensor" type="imu">
+            <always_on>true</always_on>
+            <update_rate>100</update_rate>
+            <visualize>true</visualize>
+            <topic>__default_topic__</topic>
+            <plugin filename="libgazebo_ros_imu_sensor.so" name="imu_plugin">
+                <topicName>imu</topicName>
+                <bodyName>link_torso</bodyName>
+                <updateRateHZ>10.0</updateRateHZ>
+                <gaussianNoise>0.0</gaussianNoise>
+                <xyzOffset>0 0 0</xyzOffset>
+                <rpyOffset>0 0 0</rpyOffset>
+                <frameName>link_torso</frameName>
+                <initialOrientationAsReference>false</initialOrientationAsReference>
+            </plugin>
+            <pose>0 0 0 0 0 0</pose>
+            </sensor>
+        </gazebo>
+    </xacro:macro>
 </robot>

File: humanoide_gazebo/urdf/motores.xacro (robot description, xacro)
@@ -6,5 +6,5 @@
             <type>transmission_interface/SimpleTransmission</type>
             <actuator name="${motor_name}">
-                <mechanicalReduction>10</mechanicalReduction>
+                <mechanicalReduction>1</mechanicalReduction>
                 <hardwareInterface>EffortJointInterface</hardwareInterface>
             </actuator>
@@ -19,5 +19,5 @@
             <type>transmission_interface/SimpleTransmission</type>
             <actuator name="${motor_name}">
-                <mechanicalReduction>10</mechanicalReduction>
+                <mechanicalReduction>1</mechanicalReduction>
                 <hardwareInterface>EffortJointInterface</hardwareInterface>
             </actuator>
